File: enclosure/powerbrain/powerbrain.brd (EAGLE design)
At the start: 24.8 x 64.8 mm, 43 parts, among them Q2 200mA/50V, X2 ZX62D-B-5PA8

Commit message: powerbrain: ready for ordering
Parts:
- BL1: device SparkFun-Passives:B82462G -> SparkFun-Passives:SRU5028
- moved J2 5.08 mm to (22.2, 39.4)
- moved SH2 2.84 mm to (6.99, 41.6)
- moved R3 1.91 mm to (14.6, 38.1)
- moved BL1 1.42 mm to (17.8, 50.2), turned to 180 degrees
Connections:
- net BATT_VCC: now also BL1.2; no longer BL1.P$2
- net B_SW: now also BL1.1; no longer BL1.P$1
Routing:
- net GND: track 86.3 -> 94.4 mm
- net RX: track 23.2 -> 28.8 mm
- net TX: track 24.2 -> 29.3 mm
- net VCC: track 100.3 -> 98.6 mm
- net BATT_VCC: track 44.6 -> 46.0 mm
- net N$6: track 6.57 -> 6.01 mm
Other:
- board text added: "TX"
- board text removed: "select coil size"
