File: enclosure/powerbrain2/powerbrain2.brd (EAGLE design)
At the start: 24.8 x 64.8 mm, 45 parts, among them Q2 200mA/50V, Q3 200mA/50V, X2 ZX62D-B-5PA8

Commit message: powerbrain
Parts:
- moved C5 0.63 mm to (13.3, 10.2)
- moved Y1 0.31 mm to (18.1, 11.2)
Routing:
- net N$9: track 8.33 -> 9.08 mm
Changed lines of the file:
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@@
 <setting verticaltext="up"/>
 </settings>
-<grid distance="0.025" unitdist="inch" unit="inch" style="lines" multiple="1" display="yes" altdistance="0.001" altunitdist="inch" altunit="inch"/>
+<grid distance="0.025" unitdist="inch" unit="inch" style="dots" multiple="1" display="yes" altdistance="0.001" altunitdist="inch" altunit="inch"/>
 <layers>
 <layer number="1" name="Top" color="4" fill="1" visible="yes" active="yes"/>
@@
 </element>
 <element name="C4" library="SparkFun-Passives" package="1206" value="22pF" x="22.7584" y="10.795" smashed="yes" rot="R90"/>
-<element name="C5" library="SparkFun-Passives" package="1206" value="22pF" x="13.97" y="10.16" smashed="yes" rot="R90"/>
+<element name="C5" library="SparkFun-Passives" package="1206" value="22pF" x="13.335" y="10.16" smashed="yes" rot="R90"/>
 <element name="C3" library="SparkFun-Passives" package="1206" value="10uF" x="8.89" y="27.305" smashed="yes"/>
-<element name="Y1" library="SparkFun-FreqCtrl" package="CRYSTAL-SMD-5X3" value="" x="18.415" y="11.176" smashed="yes">
-<attribute name="PROD_ID" value="XTAL-08218" x="18.415" y="11.176" size="1.778" layer="27" display="off"/>
-<attribute name="VALUE" x="13.335" y="7.239" size="1.27" layer="27" ratio="10"/>
+<element name="Y1" library="SparkFun-FreqCtrl" package="CRYSTAL-SMD-5X3" value="" x="18.1102" y="11.1506" smashed="yes">
+<attribute name="PROD_ID" value="XTAL-08218" x="18.1102" y="11.1506" size="1.778" layer="27" display="off"/>
+<attribute name="VALUE" x="13.0302" y="7.2136" size="1.27" layer="27" ratio="10"/>
 </element>
 <element name="X2" library="zx62d-b-5pa8-oshpark_10" package="ZX62D-B-5PA8" value="ZX62D-B-5PA8" x="0" y="21.59" smashed="yes">
@@
 <wire x1="10.29" y1="27.305" x2="10.16" y2="27.175" width="0.254" layer="1"/>
 <via x="6.985" y="17.78" extent="1-16" drill="0.35"/>
-<wire x1="13.97" y1="8.76" x2="13.97" y2="8.4328" width="0.254" layer="1"/>
+<wire x1="13.335" y1="8.76" x2="13.97" y2="8.4328" width="0.254" layer="1"/>
 <wire x1="2.503" y1="15.203" x2="2.503" y2="14.935" width="0.254" layer="1"/>
 <wire x1="4.825" y1="20.29" x2="6.38" y2="20.29" width="0.4064" layer="1"/>
@@
 <contactref element="C4" pad="2"/>
 <contactref element="Y1" pad="3"/>
-<wire x1="20.059" y1="12.326" x2="20.265" y2="12.326" width="0.254" layer="1"/>
+<wire x1="20.059" y1="12.326" x2="19.9602" y2="12.3006" width="0.254" layer="1"/>
 <wire x1="20.059" y1="12.326" x2="19.05" y2="13.335" width="0.254" layer="1"/>
 <wire x1="19.05" y1="13.335" x2="17.78" y2="13.335" width="0.254" layer="1"/>
 <wire x1="17.78" y1="13.335" x2="17.145" y2="13.97" width="0.254" layer="1"/>
 <wire x1="17.145" y1="13.97" x2="17.145" y2="15.79" width="0.254" layer="1"/>
-<wire x1="20.265" y1="12.326" x2="20.396" y2="12.195" width="0.254" layer="1"/>
+<wire x1="19.9602" y1="12.3006" x2="20.396" y2="12.195" width="0.254" layer="1"/>
 <wire x1="20.396" y1="12.195" x2="22.7584" y2="12.195" width="0.254" layer="1"/>
 </signal>
@@
 <contactref element="C5" pad="2"/>
 <contactref element="Y1" pad="1"/>
-<wire x1="16.345" y1="14.57" x2="16.345" y2="14.605" width="0.254" layer="1"/>
-<wire x1="16.345" y1="14.605" x2="16.345" y2="15.79" width="0.254" layer="1"/>
-<wire x1="16.565" y1="10.026" x2="16.139" y2="10.026" width="0.254" layer="1"/>
-<wire x1="13.97" y1="11.56" x2="16.139" y2="10.026" width="0.254" layer="1"/>
-<wire x1="16.345" y1="14.605" x2="16.345" y2="14.44" width="0.254" layer="1"/>
+<wire x1="16.345" y1="14.44" x2="16.345" y2="15.79" width="0.254" layer="1"/>
+<wire x1="16.2602" y1="10.0006" x2="14.869" y2="10.026" width="0.254" layer="1"/>
+<wire x1="13.335" y1="11.56" x2="14.869" y2="10.026" width="0.254" layer="1"/>
 <wire x1="16.345" y1="14.44" x2="13.97" y2="12.065" width="0.254" layer="1"/>
-<wire x1="13.97" y1="12.065" x2="13.97" y2="11.56" width="0.254" layer="1"/>
+<wire x1="13.97" y1="12.065" x2="13.335" y2="11.56" width="0.254" layer="1"/>
 </signal>
 <signal name="VBUS_SENSE">

Commit message: powerbrain2 sent to fab
Parts:
- removed BC1: 10uF, SparkFun-Capacitors:1206
- removed BC2: 2.2uF, SparkFun-Capacitors:1206
- removed BL1: 6.8uH / 2A, SparkFun-Passives:SRU5028
- removed BR1, BR3: 1.87M, SparkFun-Resistors:1206
- removed BR2: 340k, SparkFun-Resistors:1206
- removed BR4: 200k, SparkFun-Resistors:1206
- removed BR5: (no value), SparkFun-Resistors:1206
- removed C7: 100uF / 6V, SparkFun-Passives:EIA3528-KIT
- removed H4: MOUNT-HOLE2.8, holes:2,8
- removed U2: (no value), TPS61090:QFN65P400X400X100-17N
- added J5: (no value), SparkFun-Connectors:1X03_LOCK
- moved SH2 6.98 mm to (12.5, 45.9), turned to 0 degrees
- moved J2 3.81 mm to (22.2, 35.6)
- moved R3 1.27 mm to (14.6, 36.8)
- moved J1 0.90 mm to (9.53, 45.7)
- moved J4 0.63 mm to (2.54, 45.7)
Connections:
- removed net B_FB: BR3.2, BR4.1, U2.14
- removed net B_LBI: BR1.1, BR2.2, U2.9
- removed net B_SW: BL1.1, U2.3, U2.4
- removed net LOW_BATTERY_OUTPUT: BR5.2, U2.12
- net BATT_GND: no longer BC1.2, BC2.1, BR2.1, BR4.2, C7.C, U2.10, U2.13, U2.17, U2.5, U2.6, U2.7, U2.P$1
- net BATT_VCC: now also J5.3; no longer BC1.1, BL1.2, BR1.2, U2.11, U2.8
- net GND: now also J5.2
- net VCC: now also J5.1; no longer BC2.2, BR3.1, BR5.1, C7.A, U2.1, U2.15, U2.16
Routing:
- net BATT_GND: track 37.7 -> 9.29 mm
- net BATT_VCC: track 46.0 -> 27.1 mm, vias 3 -> 0
- net LOW_BATTERY_OUTPUT: track 15.9 -> 0.00 mm
- net VCC: track 98.6 -> 86.5 mm
- net GND: track 94.8 -> 86.5 mm
- net B_FB: track 7.41 -> 0.00 mm
- net B_LBI: track 7.30 -> 0.00 mm
- net RX: track 28.8 -> 25.0 mm
- net TX: track 29.3 -> 25.4 mm
- removed copper zone on layer 1, net BATT_GND
- removed copper zone on layer 16, net BATT_GND
- removed copper zone on layer 1, net BATT_VCC
- removed copper zone on layer 1, net B_SW
- removed copper zone on layer 1, net VCC
Other:
- board size 24.8 x 64.8 mm -> 24.8 x 48.3 mm
- board text added: "B"
- board text added: "V"

Commit message: cleaned up the powerbrain2 schematics
Connections:
- removed net CAM1: U$3.28
- removed net CAM2: U$3.27
- removed net CAM3: U$3.26
- removed net CAM4: U$3.25
- removed net FOO2: U$3.30
- removed net FOO3: U$3.8
- removed net FOO4: U$3.37
- removed net FOO5: U$3.22
- removed net FOO6: U$3.29
- removed net FOO7: U$3.32
- removed net FOO8: U$3.39
Changed lines of the file:
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@@
 <wire x1="22.2504" y1="16.4846" x2="22.86" y2="15.875" width="0.254" layer="16"/>
-</signal>
-<signal name="CAM1">
-<contactref element="U$3" pad="28"/>
-</signal>
-<signal name="CAM2">
-<contactref element="U$3" pad="27"/>
 </signal>
 <signal name="BATT_VCC" class="2">
@@
 <wire x1="16.9418" y1="29.0576" x2="16.9418" y2="30.48" width="0.254" layer="1"/>
 </signal>
-<signal name="CAM3">
-<contactref element="U$3" pad="26"/>
-</signal>
-<signal name="CAM4">
-<contactref element="U$3" pad="25"/>
-</signal>
 <signal name="USB_VCC">
 <contactref element="Q1" pad="3"/>
@@
 <wire x1="2.54" y1="34.925" x2="2.54" y2="31.75" width="0.762" layer="16"/>
 </signal>
-<signal name="FOO3">
-<contactref element="U$3" pad="8"/>
-</signal>
-<signal name="FOO6">
-<contactref element="U$3" pad="29"/>
-</signal>
 <signal name="CAM_EN">
 <contactref element="U$3" pad="31"/>
-</signal>
-<signal name="FOO4">
-<contactref element="U$3" pad="37"/>
-</signal>
-<signal name="FOO8">
-<contactref element="U$3" pad="39"/>
-</signal>
-<signal name="FOO5">
-<contactref element="U$3" pad="22"/>
 </signal>
 <signal name="N$6">
@@
 <wire x1="19.685" y1="30.5816" x2="19.685" y2="30.985" width="0.254" layer="1"/>
 </signal>
-<signal name="FOO2">
-<contactref element="U$3" pad="30"/>
-</signal>
-<signal name="FOO7">
-<contactref element="U$3" pad="32"/>
-</signal>
 <signal name="$N23">
